File: WachcioDrop/WachcioDrop/Shift_registers.kicad_sch (KiCad schematic)
At the start: 61 parts, among them J1 Conn_01x10_Socket, K10 G3MB-202P, K2 G3MB-202P, K3 G3MB-202P, K4 G3MB-202P, K5 G3MB-202P, K6 G3MB-202P, K7 G3MB-202P, K8 G3MB-202P, K9 G3MB-202P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

Commit message: 20_04_2026
Parts:
- R1, R10, R13, R16, R19, R22, R25, R28, R29, R4, R7: value 150R -> 270R
- R11, R14, R17, R2, R20, R23, R26, R5, R8: value 10K -> 4,7K
Changed lines of the file:
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@@
 			)
 		)
-		(property "Value" "10K"
+		(property "Value" "4,7K"
 			(at 184.15 57.15 90)
 			(show_name no)
@@
 			)
 		)
-		(property "Value" "10K"
+		(property "Value" "4,7K"
 			(at 22.86 57.15 90)
 			(show_name no)
@@
 			)
 		)
-		(property "Value" "10K"
+		(property "Value" "4,7K"
 			(at 226.06 57.15 90)
 			(show_name no)
@@
 			)
 		)
-		(property "Value" "10K"
+		(property "Value" "4,7K"
 			(at 24.13 119.38 90)
 			(show_name no)
@@
 			)
 		)
-		(property "Value" "150R"
+		(property "Value" "270R"
 			(at 184.912 48.26 90)
 			(show_name no)
@@
 			)
 		)
-		(property "Value" "150R"
+		(property "Value" "270R"
 			(at 62.992 48.26 90)
 			(show_name no)
@@
 			)
 		)
-		(property "Value" "10K"
+		(property "Value" "4,7K"
 			(at 66.04 119.38 90)
 			(show_name no)
@@
 			)
 		)
-		(property "Value" "150R"
+		(property "Value" "270R"
 			(at 66.802 110.49 90)
 			(show_name no)
@@
 			)
 		)
-		(property "Value" "10K"
+		(property "Value" "4,7K"
 			(at 62.23 57.15 90)
 			(show_name no)
@@
 			)
 		)
-		(property "Value" "150R"
+		(property "Value" "270R"
 			(at 173.99 113.792 90)
 			(show_name no)
@@
 			)
 		)
-		(property "Value" "150R"
+		(property "Value" "270R"
 			(at 24.892 110.49 90)
 			(show_name no)
@@
 			)
 		)
-		(property "Value" "150R"
+		(property "Value" "270R"
 			(at 226.822 48.26 90)
 			(show_name no)
@@
 			)
 		)
-		(property "Value" "150R"
+		(property "Value" "270R"
 			(at 23.622 48.26 90)
 			(show_name no)
@@
 			)
 		)
-		(property "Value" "150R"
+		(property "Value" "270R"
 			(at 182.88 113.792 90)
 			(show_name no)
@@
 			)
 		)
-		(property "Value" "150R"
+		(property "Value" "270R"
 			(at 107.442 110.49 90)
 			(show_name no)
@@
 			)
 		)
-		(property "Value" "150R"
+		(property "Value" "270R"
 			(at 103.632 48.26 90)
 			(show_name no)
@@
 			)
 		)
-		(property "Value" "150R"
+		(property "Value" "270R"
 			(at 144.272 48.26 90)
 			(show_name no)
@@
 			)
 		)
-		(property "Value" "10K"
+		(property "Value" "4,7K"
 			(at 106.68 119.38 90)
 			(show_name no)
@@
 			)
 		)
-		(property "Value" "10K"
+		(property "Value" "4,7K"
 			(at 143.51 57.15 90)
 			(show_name no)
@@
 			)
 		)
-		(property "Value" "10K"
+		(property "Value" "4,7K"
 			(at 102.87 57.15 90)
 			(show_name no)
