File: WachcioDrop/WachcioDrop/WachcioDrop.kicad_sch (KiCad schematic)
At the start: 3 parts, among them K1 G3MB-202P, U1 ESP32-S3-DEVKITC-1-N8R2, U3 TC00500

Commit message: 20_04_2026
Parts:
- removed K1: G3MB-202P, G3MB-202P:RELAY_G3MB-202P, symbol Wachcio:G3MB-202P
