File: WachcioDrop/WachcioDrop_kopia/Shift_registers.kicad_sch (KiCad schematic)
At the start: 61 parts, among them J1 Conn_01x10_Socket, K1 G3MB-202P, K2 G3MB-202P, K3 G3MB-202P, K4 G3MB-202P, K5 G3MB-202P, K6 G3MB-202P, K7 G3MB-202P, K8 G3MB-202P, K9 G3MB-202P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

Commit message: 26_04_2026
Connections:
- net section1_LED_K renamed sekcja1_LED_K
- net section2 renamed sekcja2
- net section2_LED_A renamed sekcja2_LED_A
- net section2_LED_K renamed sekcja2_LED_K
- net section3 renamed sekcja3
- net section3_LED_A renamed sekcja3_LED_A
- net section3_LED_K renamed sekcja3_LED_K
- net section4 renamed sekcja4
- net section4_LED_A renamed sekcja4_LED_A
- net section4_LED_K renamed sekcja4_LED_K
- net section5 renamed sekcja5
- net section5_LED_A renamed sekcja5_LED_A
- net section5_LED_K renamed sekcja5_LED_K
- net section6 renamed sekcja6
- net section6_LED_A renamed sekcja6_LED_A
- net section6_LED_K renamed sekcja6_LED_K
- net section7 renamed sekcja7
- net section7_LED_A renamed sekcja7_LED_A
- net section7_LED_K renamed sekcja7_LED_K
- net section8 renamed sekcja8
- net section8_LED_A renamed sekcja8_LED_A
- net section8_LED_K renamed sekcja8_LED_K
Changed lines of the file:
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@@
 		)
 	)
-	(label "section4"
+	(label "sekcja4"
 		(at 177.8 60.96 90)
 		(effects
@@
 		)
 	)
-	(label "section2"
+	(label "sekcja2"
 		(at 96.52 60.96 90)
 		(effects
@@
 		)
 	)
-	(label "section8"
+	(label "sekcja8"
 		(at 214.63 143.51 180)
 		(effects
@@
 		)
 	)
-	(label "section5_LED_K"
+	(label "sekcja5_LED_K"
 		(at 247.65 50.8 90)
 		(effects
@@
 		)
 	)
-	(label "section4_LED_K"
+	(label "sekcja4_LED_K"
 		(at 205.74 50.8 90)
 		(effects
@@
 		)
 	)
-	(label "section6_LED_A"
+	(label "sekcja6_LED_A"
 		(at 29.21 124.46 180)
 		(effects
@@
 		)
 	)
-	(label "section6_LED_K"
+	(label "sekcja6_LED_K"
 		(at 44.45 123.19 90)
 		(effects
@@
 		)
 	)
-	(label "section5"
+	(label "sekcja5"
 		(at 147.32 132.08 180)
 		(effects
@@
 		)
 	)
-	(label "section4"
+	(label "sekcja4"
 		(at 147.32 134.62 180)
 		(effects
@@
 		)
 	)
-	(label "section6"
+	(label "sekcja6"
 		(at 147.32 129.54 180)
 		(effects
@@
 		)
 	)
-	(label "section5_LED_A"
+	(label "sekcja5_LED_A"
 		(at 232.41 52.07 180)
 		(effects
@@
 		)
 	)
-	(label "section6"
+	(label "sekcja6"
 		(at 15.24 135.89 90)
 		(effects
@@
 		)
 	)
-	(label "section7"
+	(label "sekcja7"
 		(at 58.42 135.89 90)
 		(effects
@@
 		)
 	)
-	(label "section2_LED_K"
+	(label "sekcja2_LED_K"
 		(at 124.46 50.8 90)
 		(effects
@@
 		)
 	)
-	(label "section7_LED_A"
+	(label "sekcja7_LED_A"
 		(at 71.12 124.46 180)
 		(effects
@@
 		)
 	)
-	(label "section3"
+	(label "sekcja3"
 		(at 137.16 60.96 90)
 		(effects
@@
 		)
 	)
-	(label "section3"
+	(label "sekcja3"
 		(at 147.32 137.16 180)
 		(effects
@@
 		)
 	)
-	(label "section4_LED_A"
+	(label "sekcja4_LED_A"
 		(at 190.5 52.07 180)
 		(effects
@@
 		)
 	)
-	(label "section3_LED_K"
+	(label "sekcja3_LED_K"
 		(at 165.1 49.53 90)
 		(effects
@@
 		)
 	)
-	(label "section5"
+	(label "sekcja5"
 		(at 219.71 60.96 90)
 		(effects
@@
 		)
 	)
-	(label "section7"
+	(label "sekcja7"
 		(at 147.32 127 180)
 		(effects
@@
 		)
 	)
-	(label "section7_LED_K"
+	(label "sekcja7_LED_K"
 		(at 86.36 123.19 90)
 		(effects
@@
 		)
 	)
-	(label "section8_LED_A"
+	(label "sekcja8_LED_A"
 		(at 111.76 124.46 180)
 		(effects
@@
 		)
 	)
-	(label "section2"
+	(label "sekcja2"
 		(at 147.32 139.7 180)
 		(effects
@@
 		)
 	)
-	(label "section8_LED_K"
+	(label "sekcja8_LED_K"
 		(at 127 123.19 90)
 		(effects
@@
 		)
 	)
-	(label "section1_LED_K"
+	(label "sekcja1_LED_K"
 		(at 83.82 45.72 90)
 		(effects
@@
 		)
 	)
-	(label "section2_LED_A"
+	(label "sekcja2_LED_A"
 		(at 109.22 52.07 180)
 		(effects
@@
 		)
 	)
-	(label "section8"
+	(label "sekcja8"
 		(at 99.06 135.89 90)
 		(effects
@@
 		)
 	)
-	(label "section3_LED_A"
+	(label "sekcja3_LED_A"
 		(at 149.86 52.07 180)
 		(effects
