File: WachcioDrop/WachcioDrop_kopia/WachcioDrop.kicad_sch (KiCad schematic)
At the start: 3 parts, among them J2 Conn_02x20_Top_Bottom, U1 ESP32-S3-DEVKITC-1-N8R2, U2 TC00500 RTC DS3231

Commit message: 26_04_2026
Connections:
- net section1_LED_K renamed sekcja1_LED_K
- net section2_LED_A renamed sekcja2_LED_A
- net section2_LED_K renamed sekcja2_LED_K
- net section3_LED_A renamed sekcja3_LED_A
- net section3_LED_K renamed sekcja3_LED_K
- net section4_LED_A renamed sekcja4_LED_A
- net section4_LED_K renamed sekcja4_LED_K
- net section5_LED_A renamed sekcja5_LED_A
- net section5_LED_K renamed sekcja5_LED_K
- net section6_LED_A renamed sekcja6_LED_A
- net section6_LED_K renamed sekcja6_LED_K
- net section7_LED_A renamed sekcja7_LED_A
- net section7_LED_K renamed sekcja7_LED_K
- net section8_LED_A renamed sekcja8_LED_A
- net section8_LED_K renamed sekcja8_LED_K
Changed lines of the file:
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@@
 		)
 	)
-	(label "section7_LED_A"
+	(label "sekcja7_LED_A"
 		(at 166.37 50.8 0)
 		(effects
@@
 		)
 	)
-	(label "section1_LED_K"
+	(label "sekcja1_LED_K"
 		(at 143.51 45.72 180)
 		(effects
@@
 		)
 	)
-	(label "section2_LED_K"
+	(label "sekcja2_LED_K"
 		(at 143.51 50.8 180)
 		(effects
@@
 		)
 	)
-	(label "section4_LED_K"
+	(label "sekcja4_LED_K"
 		(at 143.51 60.96 180)
 		(effects
@@
 		)
 	)
-	(label "section4_LED_A"
+	(label "sekcja4_LED_A"
 		(at 143.51 58.42 180)
 		(effects
@@
 		)
 	)
-	(label "section2_LED_A"
+	(label "sekcja2_LED_A"
 		(at 143.51 48.26 180)
 		(effects
@@
 		)
 	)
-	(label "section3_LED_K"
+	(label "sekcja3_LED_K"
 		(at 143.51 55.88 180)
 		(effects
@@
 		)
 	)
-	(label "section7_LED_K"
+	(label "sekcja7_LED_K"
 		(at 166.37 53.34 0)
 		(effects
@@
 		)
 	)
-	(label "section6_LED_A"
+	(label "sekcja6_LED_A"
 		(at 166.37 45.72 0)
 		(effects
@@
 		)
 	)
-	(label "section8_LED_K"
+	(label "sekcja8_LED_K"
 		(at 166.37 58.42 0)
 		(effects
@@
 		)
 	)
-	(label "section6_LED_K"
+	(label "sekcja6_LED_K"
 		(at 166.37 48.26 0)
 		(effects
@@
 		)
 	)
-	(label "section8_LED_A"
+	(label "sekcja8_LED_A"
 		(at 166.37 55.88 0)
 		(effects
@@
 		)
 	)
-	(label "section5_LED_A"
+	(label "sekcja5_LED_A"
 		(at 166.37 40.64 0)
 		(effects
@@
 		)
 	)
-	(label "section5_LED_K"
+	(label "sekcja5_LED_K"
 		(at 166.37 43.18 0)
 		(effects
@@
 		)
 	)
-	(label "section3_LED_A"
+	(label "sekcja3_LED_A"
 		(at 143.51 53.34 180)
 		(effects
